Commit message: Fix jingchu03 fixed-base training stability

File: assets/jingchu03/urdf_jc01.urdf (robot description, URDF)
Before this commit: robot JingChu01, 19 links, 18 joints
Joints:
- joint left_elbow_pitch: limit lower=0 upper=1.7976 effort=0 velocity=0 -> lower=0 upper=1.7976 effort=80 velocity=20
- joint left_elbow_yaw: limit lower=-1.9722 upper=1.9722 effort=0 velocity=0 -> lower=-1.9722 upper=1.9722 effort=80 velocity=20
- joint left_shoulder_pitch: limit lower=-1.0122 upper=3.1066 effort=0 velocity=0 -> lower=-1.0122 upper=3.1066 effort=100 velocity=20
- joint left_shoulder_roll: limit lower=-0.0523 upper=2.2340 effort=0 velocity=0 -> lower=-0.0523 upper=2.2340 effort=100 velocity=20
- joint left_shoulder_yaw: limit lower=-1.9722 upper=1.9722 effort=0 velocity=0 -> lower=-1.9722 upper=1.9722 effort=100 velocity=20
- joint left_wrist_pitch: limit lower=-1.047 upper=1.047 effort=0 velocity=0 -> lower=-1.047 upper=1.047 effort=60 velocity=20
- joint left_wrist_roll: limit lower=-1.047 upper=1.047 effort=0 velocity=0 -> lower=-1.047 upper=1.047 effort=60 velocity=20
- joint right_elbow_pitch: limit lower=0 upper=1.7976 effort=0 velocity=0 -> lower=0 upper=1.7976 effort=80 velocity=20
- joint right_elbow_yaw: limit lower=-1.9722 upper=1.9722 effort=0 velocity=0 -> lower=-1.9722 upper=1.9722 effort=80 velocity=20
- joint right_shoulder_pitch: limit lower=-1.0122 upper=3.1066 effort=0 velocity=0 -> lower=-1.0122 upper=3.1066 effort=100 velocity=20
- joint right_shoulder_roll: limit lower=-0.0523 upper=2.2340 effort=0 velocity=0 -> lower=-0.0523 upper=2.2340 effort=100 velocity=20
- joint right_shoulder_yaw: limit lower=-1.9722 upper=1.9722 effort=0 velocity=0 -> lower=-1.9722 upper=1.9722 effort=100 velocity=20
- joint right_wrist_pitch: limit lower=-1.047 upper=1.047 effort=0 velocity=0 -> lower=-1.047 upper=1.047 effort=60 velocity=20
- joint right_wrist_roll: limit lower=-1.047 upper=1.047 effort=0 velocity=0 -> lower=-1.047 upper=1.047 effort=60 velocity=20
- joint waist_roll: limit lower=-0.2617 upper=0.2617 effort=0 velocity=0 -> lower=-0.2617 upper=0.2617 effort=150 velocity=20
- joint waist_yaw: limit lower=-0.7853 upper=0.7853 effort=0 velocity=0 -> lower=-0.7853 upper=0.7853 effort=150 velocity=20
